File: RatDistortion.brd (EAGLE design)
At the start: 100 x 80 mm, 40 parts, among them IC1 LM308D, J1 696103201002

Commit message: Update schemetic
Parts:
- added JN1: 2N5458, 2N5458:TO92
- added VR1, VR2, VR3: PTV09A-4225F-B104, PTV09A-4225F-B104:PTV09
Connections:
- removed net N$15: C11.1, R10.2
- new net OUTSTAGE: C11.1, C12.1, R10.2
- net 9V: now also JN1.3
- net GND: now also VR3.1
- net N$16: now also VR2.1
- net N$17: now also JN1.2
- net N$18: now also VR3.3
- net N$20: now also VR3.2
- net N$5: now also VR1.2, VR1.3
- net N$6: now also VR1.1
- net N$8: now also JN1.1
- net TONE: now also VR2.2, VR2.3
Changed lines of the file:
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@@
 <element name="JP7" library="adafruit" library_urn="urn:adsk.eagle:library:420" package="1X1-BIGPOGO" package3d_urn="urn:adsk.eagle:package:6240953/1" value="" x="-45.72" y="-44.45" smashed="yes"/>
 <element name="JP8" library="adafruit" library_urn="urn:adsk.eagle:library:420" package="1X1-BIGPOGO" package3d_urn="urn:adsk.eagle:package:6240953/1" value="" x="-45.72" y="-48.26" smashed="yes"/>
+<element name="VR1" library="PTV09A-4225F-B104" package="PTV09" value="PTV09A-4225F-B104" x="-55.88" y="-48.26" smashed="yes">
+<attribute name="AVAILABILITY" value="In Stock" x="-55.88" y="-48.26" size="1.778" layer="27" display="off"/>
+<attribute name="DESCRIPTION" value=" 100k Ohm 1 Gang Linear Through Hole, Snap In Potentiometer Detent 1.0 Kierros Carbon 0.05W, 1/20W PC Pins, Board Locks " x="-55.88" y="-48.26" size="1.778" layer="27" display="off"/>
+<attribute name="MF" value="Bourns" x="-55.88" y="-48.26" size="1.778" layer="27" display="off"/>
+<attribute name="MP" value="PTV09A-4225F-B104" x="-55.88" y="-48.26" size="1.778" layer="27" display="off"/>
+<attribute name="NAME" x="-58.88" y="-34.26" size="1.27" layer="25"/>
+<attribute name="PACKAGE" value="None" x="-55.88" y="-48.26" size="1.778" layer="27" display="off"/>
+<attribute name="PRICE" value="None" x="-55.88" y="-48.26" size="1.778" layer="27" display="off"/>
+<attribute name="PURCHASE-URL" value="https://pricing.snapeda.com/search/part/PTV09A-4225F-B104/?ref=eda" x="-55.88" y="-48.26" size="1.778" layer="27" display="off"/>
+<attribute name="VALUE" x="-58.88" y="-38.26" size="1.27" layer="27"/>
+</element>
+<element name="VR2" library="PTV09A-4225F-B104" package="PTV09" value="PTV09A-4225F-B104" x="-68.58" y="-48.26" smashed="yes">
+<attribute name="AVAILABILITY" value="In Stock" x="-68.58" y="-48.26" size="1.778" layer="27" display="off"/>
+<attribute name="DESCRIPTION" value=" 100k Ohm 1 Gang Linear Through Hole, Snap In Potentiometer Detent 1.0 Kierros Carbon 0.05W, 1/20W PC Pins, Board Locks " x="-68.58" y="-48.26" size="1.778" layer="27" display="off"/>
+<attribute name="MF" value="Bourns" x="-68.58" y="-48.26" size="1.778" layer="27" display="off"/>
+<attribute name="MP" value="PTV09A-4225F-B104" x="-68.58" y="-48.26" size="1.778" layer="27" display="off"/>
+<attribute name="NAME" x="-71.58" y="-34.26" size="1.27" layer="25"/>
+<attribute name="PACKAGE" value="None" x="-68.58" y="-48.26" size="1.778" layer="27" display="off"/>
+<attribute name="PRICE" value="None" x="-68.58" y="-48.26" size="1.778" layer="27" display="off"/>
+<attribute name="PURCHASE-URL" value="https://pricing.snapeda.com/search/part/PTV09A-4225F-B104/?ref=eda" x="-68.58" y="-48.26" size="1.778" layer="27" display="off"/>
+<attribute name="VALUE" x="-71.58" y="-38.26" size="1.27" layer="27"/>
+</element>
+<element name="VR3" library="PTV09A-4225F-B104" package="PTV09" value="PTV09A-4225F-B104" x="-81.28" y="-48.26" smashed="yes">
+<attribute name="AVAILABILITY" value="In Stock" x="-81.28" y="-48.26" size="1.778" layer="27" display="off"/>
+<attribute name="DESCRIPTION" value=" 100k Ohm 1 Gang Linear Through Hole, Snap In Potentiometer Detent 1.0 Kierros Carbon 0.05W, 1/20W PC Pins, Board Locks " x="-81.28" y="-48.26" size="1.778" layer="27" display="off"/>
+<attribute name="MF" value="Bourns" x="-81.28" y="-48.26" size="1.778" layer="27" display="off"/>
+<attribute name="MP" value="PTV09A-4225F-B104" x="-81.28" y="-48.26" size="1.778" layer="27" display="off"/>
+<attribute name="NAME" x="-84.28" y="-34.26" size="1.27" layer="25"/>
+<attribute name="PACKAGE" value="None" x="-81.28" y="-48.26" size="1.778" layer="27" display="off"/>
+<attribute name="PRICE" value="None" x="-81.28" y="-48.26" size="1.778" layer="27" display="off"/>
+<attribute name="PURCHASE-URL" value="https://pricing.snapeda.com/search/part/PTV09A-4225F-B104/?ref=eda" x="-81.28" y="-48.26" size="1.778" layer="27" display="off"/>
+<attribute name="VALUE" x="-84.28" y="-38.26" size="1.27" layer="27"/>
+</element>
+<element name="JN1" library="2N5458" package="TO92" value="2N5458" x="-83.82" y="-53.34" smashed="yes">
+<attribute name="AVAILABILITY" value="In Stock" x="-83.82" y="-53.34" size="1.778" layer="27" display="off"/>
+<attribute name="DESCRIPTION" value=" JFET N-Channel 25 V 310 mW Through Hole TO-92 (TO-226) " x="-83.82" y="-53.34" size="1.778" layer="27" display="off"/>
+<attribute name="MF" value="ON Semiconductor" x="-83.82" y="-53.34" size="1.778" layer="27" display="off"/>
+<attribute name="MP" value="2N5458" x="-83.82" y="-53.34" size="1.778" layer="27" display="off"/>
+<attribute name="NAME" x="-80.64151875" y="-52.704303125" size="1.271390625" layer="25" ratio="10"/>
+<attribute name="PACKAGE" value="E-PKG AXIAL-LEADED-2 ON Semiconductor" x="-83.82" y="-53.34" size="1.778" layer="27" display="off"/>
+<attribute name="PRICE" value="None" x="-83.82" y="-53.34" size="1.778" layer="27" display="off"/>
+<attribute name="VALUE" x="-80.639159375" y="-54.61233125" size="1.27233125" layer="27" ratio="10"/>
+</element>
 </elements>
 <signals>
@@
 <contactref element="IC1" pad="7"/>
 <contactref element="R13" pad="2"/>
+<contactref element="JN1" pad="3"/>
+<wire x1="-46.14" y1="-40.64" x2="-85.09" y2="-53.34" width="0" layer="19" extent="1-1"/>
 <wire x1="-45.085" y1="6.41" x2="-46.14" y2="-40.64" width="0" layer="19" extent="1-1"/>
 <wire x1="-46.57" y1="25.4" x2="-45.085" y2="6.41" width="0" layer="19" extent="1-1"/>
@@
 <contactref element="R12" pad="1"/>
 <contactref element="JP8" pad="P$1"/>
+<contactref element="VR3" pad="1"/>
+<wire x1="-45.72" y1="-48.26" x2="-83.78" y2="-48.26" width="0" layer="19" extent="1-1"/>
 <wire x1="-47.84" y1="-22.86" x2="-45.72" y2="-48.26" width="0" layer="19" extent="1-1"/>
 <wire x1="-47.84" y1="-17.78" x2="-47.84" y2="-22.86" width="0" layer="19" extent="1-1"/>
@@
 <contactref element="C6" pad="1"/>
 <contactref element="IC1" pad="2"/>
+<contactref element="VR1" pad="3"/>
+<contactref element="VR1" pad="2"/>
+<wire x1="-53.38" y1="-48.26" x2="-55.88" y2="-48.26" width="0" layer="19" extent="1-1"/>
+<wire x1="-45.085" y1="1.21" x2="-53.38" y2="-48.26" width="0" layer="19" extent="1-1"/>
 <wire x1="-28.79" y1="25.4" x2="-45.085" y2="1.21" width="0" layer="19" extent="1-1"/>
 <wire x1="-30.9" y1="33.02" x2="-28.79" y2="25.4" width="0" layer="19" extent="1-1"/>
 <wire x1="-14.39" y1="38.1" x2="-30.9" y2="33.02" width="0" layer="19" extent="1-1"/>
-</signal>
-<signal name="N$6">
-<contactref element="C6" pad="2"/>
 </signal>
 <signal name="N$7">
@@
 <contactref element="D2" pad="C"/>
 <contactref element="D3" pad="A"/>
-<wire x1="-33.02" y1="39.37" x2="-18.2" y2="38.1" width="0" layer="19" extent="1-1"/>
-<wire x1="-36.83" y1="39.37" x2="-33.02" y2="39.37" width="0" layer="19" extent="1-1"/>
+<contactref element="VR2" pad="2"/>
+<contactref element="VR2" pad="3"/>
+<wire x1="-66.08" y1="-48.26" x2="-68.58" y2="-48.26" width="0" layer="19" extent="1-1"/>
+<wire x1="-36.83" y1="39.37" x2="-66.08" y2="-48.26" width="0" layer="19" extent="1-1"/>
+<wire x1="-33.02" y1="39.37" x2="-36.83" y2="39.37" width="0" layer="19" extent="1-1"/>
+<wire x1="-18.2" y1="38.1" x2="-33.02" y2="39.37" width="0" layer="19" extent="1-1"/>
 </signal>
 <signal name="N$9">
@@
 <wire x1="-41.06" y1="33.02" x2="-27.52" y2="33.02" width="0" layer="19" extent="1-1"/>
 </signal>
-<signal name="N$15">
+<signal name="OUTSTAGE">
 <contactref element="R10" pad="2"/>
 <contactref element="C11" pad="1"/>
+<contactref element="C12" pad="1"/>
+<wire x1="-47.84" y1="-7.62" x2="-47.84" y2="-12.7" width="0" layer="19" extent="1-1"/>
 <wire x1="-46.14" y1="-2.54" x2="-47.84" y2="-7.62" width="0" layer="19" extent="1-1"/>
 </signal>
 <signal name="N$16">
 <contactref element="R10" pad="1"/>
+<contactref element="VR2" pad="1"/>
+<wire x1="-47.84" y1="-2.54" x2="-71.08" y2="-48.26" width="0" layer="19" extent="1-1"/>
 </signal>
 <signal name="N$8">
 <contactref element="C12" pad="2"/>
 <contactref element="R11" pad="2"/>
+<contactref element="JN1" pad="1"/>
+<wire x1="-46.14" y1="-17.78" x2="-82.55" y2="-53.34" width="0" layer="19" extent="1-1"/>
 <wire x1="-46.14" y1="-12.7" x2="-46.14" y2="-17.78" width="0" layer="19" extent="1-1"/>
 </signal>
@@
 <contactref element="C13" pad="1"/>
 <contactref element="R12" pad="2"/>
+<contactref element="JN1" pad="2"/>
+<wire x1="-47.12" y1="-29.21" x2="-83.82" y2="-51.435" width="0" layer="19" extent="1-1"/>
 <wire x1="-46.14" y1="-22.86" x2="-47.12" y2="-29.21" width="0" layer="19" extent="1-1"/>
 </signal>
 <signal name="N$18">
 <contactref element="C13" pad="2"/>
+<contactref element="VR3" pad="3"/>
+<wire x1="-44.32" y1="-29.21" x2="-78.78" y2="-48.26" width="0" layer="19" extent="1-1"/>
 </signal>
 <signal name="N$20">
 <contactref element="JP5" pad="P$1"/>
+<contactref element="VR3" pad="2"/>
+<wire x1="-35.56" y1="43.18" x2="-81.28" y2="-48.26" width="0" layer="19" extent="1-1"/>
 </signal>
 <signal name="N$19">
@@
 <wire x1="-44.45" y1="-35.56" x2="-45.72" y2="-44.45" width="0" layer="19" extent="1-1"/>
 </signal>
+<signal name="N$6">
+<contactref element="C6" pad="2"/>
+<contactref element="VR1" pad="1"/>
+<wire x1="-27.09" y1="25.4" x2="-58.38" y2="-48.26" width="0" layer="19" extent="1-1"/>
+</signal>
 </signals>

Commit message: Schemetic and PCB
Parts:
- removed J1: 696103201002, 696103201002:696103201002
- added F1: 100mA, adafruit:1812
- moved VR1 128.3 mm to (48.0, 27.0), flipped to the bottom
- moved VR2 122.0 mm to (27.5, 27.0), flipped to the bottom
- moved JN1 117.0 mm to (7.58, 19.7)
- moved VR3 116.0 mm to (7.00, 27.0), flipped to the bottom
- moved JP5 92.3 mm to (48.0, 4.00), turned to 90 degrees
- moved R13 89.3 mm to (27.5, 8.64), turned to 180 degrees
- moved C4 85.0 mm to (48.0, 34.6), turned to 270 degrees
- moved LED1 83.7 mm to (27.5, 5.00), turned to 180 degrees
- moved C5 82.4 mm to (39.0, 34.6), turned to 270 degrees
- moved JP6 81.9 mm to (40.0, 41.0), turned to 90 degrees
- moved JP1 80.8 mm to (35.0, 41.0), turned to 90 degrees
- moved JP2 78.9 mm to (52.0, 4.00), turned to 90 degrees
- moved JP7 77.7 mm to (15.0, 4.00), flipped to the bottom, turned to 270 degrees
- moved C6 77.2 mm to (49.3, 24.6)
- moved JP8 77.1 mm to (11.0, 4.00), turned to 90 degrees
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Connections:
- removed net N$11: C8.1, IC1.6
- net N$1: now also F1.2; no longer J1.2
- net N$2: now also F1.1; no longer J1.1
- net N$6: now also C8.1, IC1.6
Routing:
- net 9V: track 0.00 -> 96.1 mm, vias 0 -> 2
- net N$5: track 0.00 -> 64.9 mm
- net N$6: track 0.00 -> 54.8 mm, vias 0 -> 1
- net N$20: track 0.00 -> 54.2 mm, vias 0 -> 1
- net 4.5V: track 0.00 -> 33.9 mm, vias 0 -> 2
- net N$12: track 0.00 -> 18.0 mm
- net N$16: track 0.00 -> 17.9 mm
- net TONE: track 0.00 -> 15.3 mm
- net N$21: track 0.00 -> 11.6 mm
- net N$14: track 0.00 -> 7.81 mm
- net N$17: track 0.00 -> 6.95 mm
- net N$2: track 0.00 -> 5.91 mm
- net N$8: track 0.00 -> 5.74 mm
- net OUTSTAGE: track 0.00 -> 4.39 mm
- net N$13: track 0.00 -> 4.19 mm
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- added copper zone on layer 1, net GND
- added copper zone on layer 16, net GND
Other:
- board size 100 x 80 mm -> 55 x 45 mm
- board text added: "Distortion"
- board text added: "Filter"
- board text added: "IN+"
- board text added: "IN-"
- board text added: "LED+"
- board text added: "LED-"
- board text added: "OUT+"
- board text added: "OUT-"
- board text added: "RAT distortion By Jordy Vermeulen 5021"
- board text added: "Signature"
- board text added: "Volume"
- board text added: "inside"
- board text added: "outside"
