File: RatDistortion.sch (EAGLE design)
At the start: 40 parts, among them IC1 LM308D, J1 696103201002

Commit message: Update schemetic
Parts:
- added JN1: 2N5458, 2N5458:2N5458
- added VR1, VR2, VR3: PTV09A-4225F-B104, PTV09A-4225F-B104:PTV09A-4225F-B104
Connections:
- removed net N$15: C11.1, R10.2
- new net OUTSTAGE: C11.1, C12.1, R10.2
- net 9V: now also JN1.D
- net GND: now also VR3.1
- net N$16: now also VR2.1
- net N$17: now also JN1.S
- net N$18: now also VR3.3
- net N$20: now also VR3.2
- net N$5: now also VR1.2, VR1.3
- net N$6: now also VR1.1
- net N$8: now also JN1.G
- net TONE: now also VR2.2, VR2.3
Other:
- moved on the sheet: JP5, JP6
Changed lines of the file:
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@@
 <part name="JP8" library="adafruit" library_urn="urn:adsk.eagle:library:420" deviceset="PINHD-1X1" device="-BIGPOGO" package3d_urn="urn:adsk.eagle:package:6240953/1"/>
 <part name="GND11" library="supply1" library_urn="urn:adsk.eagle:library:371" deviceset="GND" device=""/>
+<part name="VR1" library="PTV09A-4225F-B104" deviceset="PTV09A-4225F-B104" device=""/>
+<part name="VR2" library="PTV09A-4225F-B104" deviceset="PTV09A-4225F-B104" device=""/>
+<part name="VR3" library="PTV09A-4225F-B104" deviceset="PTV09A-4225F-B104" device=""/>
+<part name="JN1" library="2N5458" deviceset="2N5458" device=""/>
 </parts>
 <sheets>
@@
 -Voltage divider (4.5 volts as virtual GND)</text>
 <text x="0" y="22.86" size="1.778" layer="91">200mA</text>
-<text x="7.62" y="-20.32" size="1.778" layer="91">
+<text x="20.32" y="-20.32" size="1.778" layer="91">
 100k pot</text>
 <text x="-53.34" y="48.26" size="1.778" layer="91">pods</text>
@@
 <attribute name="VALUE" x="-52.07" y="-55.88" size="1.778" layer="96" rot="R180"/>
 </instance>
-<instance part="JP5" gate="G$1" x="5.08" y="-139.7" smashed="yes">
-<attribute name="NAME" x="-1.27" y="-136.525" size="1.778" layer="95"/>
-<attribute name="VALUE" x="-1.27" y="-144.78" size="1.778" layer="96"/>
-</instance>
-<instance part="JP6" gate="G$1" x="5.08" y="-149.86" smashed="yes">
-<attribute name="NAME" x="-1.27" y="-146.685" size="1.778" layer="95"/>
-<attribute name="VALUE" x="-1.27" y="-154.94" size="1.778" layer="96"/>
+<instance part="JP5" gate="G$1" x="15.24" y="-147.32" smashed="yes">
+<attribute name="NAME" x="8.89" y="-144.145" size="1.778" layer="95"/>
+<attribute name="VALUE" x="8.89" y="-152.4" size="1.778" layer="96"/>
+</instance>
+<instance part="JP6" gate="G$1" x="15.24" y="-157.48" smashed="yes">
+<attribute name="NAME" x="8.89" y="-154.305" size="1.778" layer="95"/>
+<attribute name="VALUE" x="8.89" y="-162.56" size="1.778" layer="96"/>
 </instance>
 <instance part="GND4" gate="1" x="-48.26" y="-63.5" smashed="yes">
 <attribute name="VALUE" x="-50.8" y="-66.04" size="1.778" layer="96"/>
 </instance>
-<instance part="GND5" gate="1" x="-5.08" y="-152.4" smashed="yes">
-<attribute name="VALUE" x="-7.62" y="-154.94" size="1.778" layer="96"/>
+<instance part="GND5" gate="1" x="-10.16" y="-160.02" smashed="yes">
+<attribute name="VALUE" x="-12.7" y="-162.56" size="1.778" layer="96"/>
 </instance>
 <instance part="C4" gate="G$1" x="-17.78" y="-27.94" smashed="yes" rot="R90">
@@
 <instance part="GND11" gate="1" x="-35.56" y="-203.2" smashed="yes">
 <attribute name="VALUE" x="-38.1" y="-205.74" size="1.778" layer="96"/>
+</instance>
+<instance part="VR1" gate="G$1" x="15.24" y="-22.86" smashed="yes" rot="R270">
+<attribute name="NAME" x="15.24" y="-27.94" size="1.27" layer="94" rot="R270"/>
+</instance>
+<instance part="VR2" gate="G$1" x="-50.8" y="-96.52" smashed="yes" rot="R270">
+<attribute name="NAME" x="-50.8" y="-101.6" size="1.27" layer="94" rot="R270"/>
+</instance>
+<instance part="VR3" gate="G$1" x="-10.16" y="-147.32" smashed="yes" rot="R180">
+<attribute name="NAME" x="-15.24" y="-147.32" size="1.27" layer="94" rot="R180"/>
+</instance>
+<instance part="JN1" gate="G$1" x="-22.86" y="-121.92" smashed="yes" rot="R90">
+<attribute name="NAME" x="-26.670140625" y="-118.109859375" size="1.77806875" layer="95" rot="R90"/>
+<attribute name="VALUE" x="-19.046940625" y="-118.106940625" size="1.77943125" layer="96" rot="R90"/>
 </instance>
 </instances>
@@
 </segment>
 <segment>
-<wire x1="-27.94" y1="-121.92" x2="-27.94" y2="-124.46" width="0.1524" layer="91"/>
-<label x="-27.94" y="-121.92" size="1.778" layer="95"/>
+<label x="-17.78" y="-116.84" size="1.778" layer="95"/>
+<pinref part="JN1" gate="G$1" pin="D"/>
+<wire x1="-17.78" y1="-116.84" x2="-17.78" y2="-121.92" width="0.1524" layer="91"/>
 </segment>
 <segment>
@@
 <pinref part="JP6" gate="G$1" pin="1"/>
 <pinref part="GND5" gate="1" pin="GND"/>
-<wire x1="2.54" y1="-149.86" x2="-5.08" y2="-149.86" width="0.1524" layer="91"/>
-<wire x1="-5.08" y1="-149.86" x2="-10.16" y2="-149.86" width="0.1524" layer="91"/>
-<junction x="-5.08" y="-149.86"/>
-<wire x1="-10.16" y1="-149.86" x2="-10.16" y2="-142.24" width="0.1524" layer="91"/>
+<wire x1="12.7" y1="-157.48" x2="-10.16" y2="-157.48" width="0.1524" layer="91"/>
+<pinref part="VR3" gate="G$1" pin="1"/>
+<junction x="-10.16" y="-157.48"/>
 </segment>
 <segment>
@@
 <wire x1="0" y1="-22.86" x2="2.54" y2="-22.86" width="0.1524" layer="91"/>
 <wire x1="2.54" y1="-22.86" x2="5.08" y2="-22.86" width="0.1524" layer="91"/>
-<wire x1="2.54" y1="-22.86" x2="2.54" y2="-20.32" width="0.1524" layer="91"/>
 <junction x="2.54" y="-22.86"/>
-<wire x1="2.54" y1="-20.32" x2="5.08" y2="-20.32" width="0.1524" layer="91"/>
 <pinref part="IC1" gate="A" pin="-IN"/>
 <wire x1="2.54" y1="-53.34" x2="0" y2="-53.34" width="0.1524" layer="91"/>
 <wire x1="0" y1="-53.34" x2="0" y2="-35.56" width="0.1524" layer="91"/>
 <junction x="0" y="-35.56"/>
-</segment>
-</net>
-<net name="N$6" class="0">
-<segment>
-<pinref part="C6" gate="G$1" pin="2"/>
-<wire x1="10.16" y1="-33.02" x2="15.24" y2="-33.02" width="0.1524" layer="91"/>
-<wire x1="15.24" y1="-33.02" x2="15.24" y2="-22.86" width="0.1524" layer="91"/>
-<wire x1="15.24" y1="-22.86" x2="10.16" y2="-22.86" width="0.1524" layer="91"/>
+<pinref part="VR1" gate="G$1" pin="3"/>
+<pinref part="VR1" gate="G$1" pin="2"/>
+<wire x1="15.24" y1="-15.24" x2="2.54" y2="-15.24" width="0.1524" layer="91"/>
+<wire x1="2.54" y1="-15.24" x2="2.54" y2="-22.86" width="0.1524" layer="91"/>
 </segment>
 </net>
@@
 </segment>
 <segment>
-<wire x1="-55.88" y1="-96.52" x2="-53.34" y2="-96.52" width="0.1524" layer="91"/>
-<wire x1="-53.34" y1="-96.52" x2="-50.8" y2="-96.52" width="0.1524" layer="91"/>
-<wire x1="-53.34" y1="-96.52" x2="-53.34" y2="-93.98" width="0.1524" layer="91"/>
-<wire x1="-53.34" y1="-93.98" x2="-50.8" y2="-93.98" width="0.1524" layer="91"/>
-<junction x="-53.34" y="-96.52"/>
-<label x="-60.96" y="-96.52" size="1.778" layer="95"/>
+<pinref part="VR2" gate="G$1" pin="2"/>
+<pinref part="VR2" gate="G$1" pin="3"/>
+<wire x1="-50.8" y1="-88.9" x2="-60.96" y2="-88.9" width="0.1524" layer="91"/>
+<wire x1="-60.96" y1="-88.9" x2="-60.96" y2="-96.52" width="0.1524" layer="91"/>
+<wire x1="-60.96" y1="-96.52" x2="-71.12" y2="-96.52" width="0.1524" layer="91"/>
+<junction x="-60.96" y="-96.52"/>
+<label x="-71.12" y="-96.52" size="1.778" layer="95"/>
 </segment>
 </net>
@@
 </segment>
 </net>
-<net name="N$15" class="0">
+<net name="OUTSTAGE" class="0">
 <segment>
 <pinref part="R10" gate="G$1" pin="2"/>
@@
 <wire x1="-27.94" y1="-96.52" x2="-12.7" y2="-96.52" width="0.1524" layer="91"/>
 <junction x="-27.94" y="-96.52"/>
+<label x="-20.32" y="-96.52" size="1.778" layer="95"/>
+</segment>
+<segment>
+<pinref part="C12" gate="G$1" pin="1"/>
+<wire x1="-48.26" y1="-132.08" x2="-58.42" y2="-132.08" width="0.1524" layer="91"/>
+<label x="-63.5" y="-132.08" size="1.778" layer="95"/>
 </segment>
 </net>
@@
 <pinref part="R10" gate="G$1" pin="1"/>
 <wire x1="-38.1" y1="-96.52" x2="-40.64" y2="-96.52" width="0.1524" layer="91"/>
+<pinref part="VR2" gate="G$1" pin="1"/>
 </segment>
 </net>
@@
 <wire x1="-40.64" y1="-132.08" x2="-38.1" y2="-132.08" width="0.1524" layer="91"/>
 <wire x1="-38.1" y1="-132.08" x2="-38.1" y2="-134.62" width="0.1524" layer="91"/>
-<wire x1="-38.1" y1="-132.08" x2="-33.02" y2="-132.08" width="0.1524" layer="91"/>
+<wire x1="-38.1" y1="-132.08" x2="-30.48" y2="-132.08" width="0.1524" layer="91"/>
 <junction x="-38.1" y="-132.08"/>
+<wire x1="-30.48" y1="-132.08" x2="-30.48" y2="-121.92" width="0.1524" layer="91"/>
+<pinref part="JN1" gate="G$1" pin="G"/>
+<wire x1="-30.48" y1="-121.92" x2="-27.94" y2="-121.92" width="0.1524" layer="91"/>
 </segment>
 </net>
@@
 <pinref part="R12" gate="G$1" pin="2"/>
 <wire x1="-22.86" y1="-134.62" x2="-27.94" y2="-134.62" width="0.1524" layer="91"/>
-<wire x1="-27.94" y1="-134.62" x2="-27.94" y2="-132.08" width="0.1524" layer="91"/>
 <junction x="-27.94" y="-134.62"/>
+<wire x1="-27.94" y1="-134.62" x2="-27.94" y2="-124.46" width="0.1524" layer="91"/>
+<wire x1="-27.94" y1="-124.46" x2="-22.86" y2="-124.46" width="0.1524" layer="91"/>
+<pinref part="JN1" gate="G$1" pin="S"/>
+<wire x1="-22.86" y1="-124.46" x2="-22.86" y2="-121.92" width="0.1524" layer="91"/>
 </segment>
 </net>
@@
 <wire x1="-15.24" y1="-134.62" x2="-10.16" y2="-134.62" width="0.1524" layer="91"/>
 <wire x1="-10.16" y1="-134.62" x2="-10.16" y2="-137.16" width="0.1524" layer="91"/>
+<pinref part="VR3" gate="G$1" pin="3"/>
 </segment>
 </net>
@@
 <segment>
 <pinref part="JP5" gate="G$1" pin="1"/>
-<wire x1="-7.62" y1="-139.7" x2="2.54" y2="-139.7" width="0.1524" layer="91"/>
+<wire x1="-2.54" y1="-147.32" x2="12.7" y2="-147.32" width="0.1524" layer="91"/>
+<pinref part="VR3" gate="G$1" pin="2"/>
 </segment>
 </net>
@@
 </segment>
 </net>
+<net name="N$6" class="0">
+<segment>
+<pinref part="C6" gate="G$1" pin="2"/>
+<pinref part="VR1" gate="G$1" pin="1"/>
+<wire x1="10.16" y1="-33.02" x2="25.4" y2="-33.02" width="0.1524" layer="91"/>
+<wire x1="25.4" y1="-33.02" x2="25.4" y2="-22.86" width="0.1524" layer="91"/>
+</segment>
+</net>

Commit message: Schemetic and PCB
Parts:
- removed J1: 696103201002, 696103201002:696103201002
- added F1: 100mA, adafruit:PTCFUSE-1812
Connections:
- removed net N$11: C8.1, IC1.OUT
- net N$1: now also F1.2; no longer J1.2
- net N$2: now also F1.1; no longer J1.1
- net N$6: now also C8.1, IC1.OUT
Other:
- note removed: "200mA"
- note removed: "pods"
- moved on the sheet: C10, C11, C12, C13, C4, C5, C6, C7, C8, C9, D2, D3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
